Commit message: add robot

File: install/my_robot_ver3/share/my_robot_ver3/urdf/my_robot_ver3.urdf (robot description, URDF)
Before this commit: robot mobile_robot, 5 links, 4 joints
Links:
- added link Lidar_link, mass 0.01; collision cylinder length=0.05 radius=0.01; visual cylinder length=0.05 radius=0.01
- added link imu_link
Joints:
- added joint Lidar_joint: type fixed, parent base_link, child Lidar_link, origin xyz=0.0 0 0.02 rpy=0 -0.087 0, axis 1 0 0
- added joint imu_joint: type fixed, parent base_link, child imu_link, origin xyz=0.0 0 0.0 rpy=0 0 0, axis 1 0 0

Commit message: GA

File: install/my_robot_ver3/share/my_robot_ver3/urdf/my_robot_ver3.urdf (robot description, URDF)
Before this commit: robot my_robot_ver3, 7 links, 6 joints
Links:
- link Lidar_link: geometry collision cylinder length=0.009 radius=0.013; visual cylinder length=0.009 radius=0.013
Joints:
- joint Lidar_joint: origin xyz=0.0 0 0.02 rpy=0 -0.087 0 -> xyz=0.0 0 0.035 rpy=0 -0.1 0
